File: kicad/dac/dac.kicad_sch (KiCad schematic)
At the start: 37 parts, among them U1 CMOD S7, U2 NE5532, U3 NE5532, U4 LM317_TO-220

Commit message: WIP
Parts:
- C2, C5, C6, C7: value 4.7u -> 100p
Connections:
- net GND: now also C2.2, C5.2, C6.2, C7.2
- net LN: now also C2.1, R6.1; no longer C2.2
- net LP: now also R5.1
- net RN: now also C6.1, R12.1; no longer C7.2
- net RP: now also C7.1, R7.1; no longer C6.1
- net LOUT: now reaches C4.2, U2.6 (-), U2.7
Other:
- note added: "Close to the FPGA"

Commit message: Added PCB
Parts:
- added C16: 100n, Custom:C_Rect_L7.2mm_W3.0mm_P5.00mm_FKS2_FKP2_MKS2_MKP2_HandSolder, symbol Device:C
- added H1, H2, H3, H4: MountingHole, MountingHole:MountingHole_3.2mm_M3, symbol Mechanical:MountingHole
- added J1: OUTPUT, Custom:Basic RCA, symbol Connector:Conn_Coaxial_x2
- added J2: Conn_01x03_Pin, Connector_JST:JST_PH_B3B-PH-K_1x03_P2.00mm_Vertical, symbol Connector:Conn_01x03_Pin
- added J3: Conn_01x08_Pin, Connector_PinHeader_2.54mm:PinHeader_1x08_P2.54mm_Vertical, symbol Connector:Conn_01x08_Pin
- added J4: I2S_IN, Connector_JST:JST_PH_B4B-PH-K_1x04_P2.00mm_Vertical, symbol Connector:Conn_01x04_Pin
- added R15, R16, R17: 100, Custom:R_Axial_DIN0204_L3.6mm_D1.6mm_P7.62mm_Horizontal_HandSolder, symbol Device:R
- added SW1: SW_DIP_x08, Button_Switch_THT:SW_DIP_SPSTx08_Slide_6.7x21.88mm_W7.62mm_P2.54mm_LowProfile, symbol Switch:SW_DIP_x08
- C1, C10, C11, C12, C13, C14, C2, C3, C4, C5, C6, C7, C8, C9: footprint (none) -> Custom:C_Rect_L7.2mm_W3.0mm_P5.00mm_FKS2_FKP2_MKS2_MKP2_HandSolder
- C15: footprint (none) -> Capacitor_THT:CP_Radial_D8.0mm_P5.00mm
- R1, R14: value 6.8k -> 10k; footprint (none) -> Custom:R_Axial_DIN0204_L3.6mm_D1.6mm_P7.62mm_Horizontal_HandSolder
- R10, R11, R12, R13, R2, R3, R4, R5, R6, R7, R8, R9: footprint (none) -> Custom:R_Axial_DIN0204_L3.6mm_D1.6mm_P7.62mm_Horizontal_HandSolder
- U2, U3: footprint (none) -> Package_DIP:DIP-8_W7.62mm
Connections:
- net +12V: now also J2.1 (Pin_1)
- net -12V: now also J2.3 (Pin_3)
- net GND: now also C16.1, J1.3 (EXT), J2.2 (Pin_2), J4.4 (Pin_4)
- net LN: now also U1.48 (A4); no longer U1.4 (N2)
- net LOUT: now also J1.2 (IN2)
- net LP: now also U1.47 (A3); no longer U1.48 (A4)
- net RN: now also U1.27 (K14); no longer U1.5 (M2)
- net ROUT: now also C14.2, U3.6 (-), U3.7, J1.1 (IN1)
- net RP: now also U1.26 (L14); no longer U1.47 (A3)
- net at D1.1 (K), U1.24 (VU): now also C16.2, SW1.1, SW1.2, SW1.3, SW1.4, SW1.5, SW1.6, SW1.7, SW1.8
- net at U1.1 (L1): now also R15.2
- net at U1.16 (P14): now also SW1.16
- net at U1.17 (P15): now also SW1.15
- net at U1.18 (N13): now also SW1.14
- net at U1.19 (N15): now also SW1.13
- net at U1.2 (M4): now also R16.2
- net at U1.20 (N14): now also SW1.12
- net at U1.21 (M15): now also SW1.11
- net at U1.22 (M14): now also SW1.10
- net at U1.23 (L15): now also SW1.9
- net at U1.3 (M3): now also R17.2
- net at U1.40 (C5): now also J3.8 (Pin_8)
- net at U1.41 (A2): now also J3.7 (Pin_7)
- net at U1.42 (B2): now also J3.6 (Pin_6)
- net at U1.43 (B1): now also J3.5 (Pin_5)
- net at U1.44 (C1): now also J3.4 (Pin_4)
- net at U1.45 (B3): now also J3.3 (Pin_3)
- net at U1.46 (B4): now also J3.2 (Pin_2)
- net P3: now reaches U1.6 (P3)
- net P3: now also J3.1 (Pin_1)
- new net BCLK: J4.2 (Pin_2), R16.1
- new net DATA: J4.1 (Pin_1), R17.1
- new net LRCLK: J4.3 (Pin_3), R15.1
- no-connect marks 0 -> 11
Other:
- note added: "Place close to the FPGA"
- note removed: "Close to the FPGA"
- moved on the sheet: D1, D2
