File: kicad/dac-ng/dac-ng.kicad_sch (KiCad schematic)
At the start: 65 parts, among them J2 Conn_01x03_Pin, J3 Conn_01x08_Pin, J4 I2S_IN, SW1 SW_DIP_x08, U1 CMOD S7, U2 OPA1612AxD, U3 OPA1612AxD, U4 LM317_TO-220

Commit message: First run of v2.0
Parts:
- removed C10, C11, C12, C9: 100n, Custom:C_Rect_L7.2mm_W3.0mm_P5.00mm_FKS2_FKP2_MKS2_MKP2_HandSolder, symbol Device:C
- removed C13, C14, C19, C20, C21, C22, C23, C24, C5, C6, C7, C8: 680p, symbol Device:C
- removed C15: 10u, Capacitor_THT:CP_Radial_D8.0mm_P5.00mm, symbol Device:C_Polarized
- removed C17, C18, C25, C26: 180p, symbol Device:C
- removed D2, D3, D4: 1N4004, Diode_THT:D_DO-41_SOD81_P10.16mm_Horizontal, symbol Diode:1N4004
- removed J2: Conn_01x03_Pin, Connector_JST:JST_PH_B3B-PH-K_1x03_P2.00mm_Vertical, symbol Connector:Conn_01x03_Pin
- removed R10, R9: 220, Custom:R_Axial_DIN0204_L3.6mm_D1.6mm_P7.62mm_Horizontal_HandSolder, symbol Device:R
- removed R11, R12, R25, R28: 15k, symbol Device:R
- removed R13, R14, R26, R27: 1.8k, symbol Device:R
- removed R18, R19, R29, R30: 1k, symbol Device:R
- removed R20, R31: 50, symbol Device:R
- removed R21, R22, R23, R24, R5, R6, R7, R8: 2.2k, symbol Device:R
- removed U2, U3: OPA1612AxD, symbol Amplifier_Operational:OPA1612AxD
- removed U4: LM317_TO-220, Package_TO_SOT_THT:TO-220-3_Vertical, symbol Regulator_Linear:LM317_TO-220
- added C2, C3: 100n, Capacitor_SMD:C_0603_1608Metric_Pad1.08x0.95mm_HandSolder, symbol Device:C
- added D1: CDBU70, Diode_SMD:D_0603_1608Metric, symbol Diode:SB140
- added U2, U3: 74LVC2G34, Package_TO_SOT_SMD:SOT-363_SC-70-6, symbol 74xGxx:74LVC2G34
- C1: renamed from C16; footprint Custom:C_Rect_L7.2mm_W3.0mm_P5.00mm_FKS2_FKP2_MKS2_MKP2_HandSolder -> Capacitor_SMD:C_0603_1608Metric_Pad1.08x0.95mm_HandSolder; Have_It (none) -> x
- D2: renamed from D1; value SB140 -> CDBU70; footprint Diode_THT:D_DO-41_SOD81_P10.16mm_Horizontal -> Diode_SMD:D_0603_1608Metric; Ordered (none) -> x
- H1: Ordered (none) -> x
- H2: renamed from H4; Ordered (none) -> x
- H3: renamed from H2; Ordered (none) -> x
- H4: renamed from H3; Ordered (none) -> x
- J1: renamed from J4; Have_It (none) -> x
- J2: renamed from J3; Have_It (none) -> x
- R1: renamed from R15; footprint Custom:R_Axial_DIN0204_L3.6mm_D1.6mm_P7.62mm_Horizontal_HandSolder -> Resistor_SMD:R_0603_1608Metric_Pad0.98x0.95mm_HandSolder; Have_It (none) -> x (50 ohm)
- R2: renamed from R16; footprint Custom:R_Axial_DIN0204_L3.6mm_D1.6mm_P7.62mm_Horizontal_HandSolder -> Resistor_SMD:R_0603_1608Metric_Pad0.98x0.95mm_HandSolder; Have_It (none) -> x (50 ohm)
- R3: renamed from R17; footprint Custom:R_Axial_DIN0204_L3.6mm_D1.6mm_P7.62mm_Horizontal_HandSolder -> Resistor_SMD:R_0603_1608Metric_Pad0.98x0.95mm_HandSolder; Have_It (none) -> x (50 ohm)
- SW1, U1: Have_It (none) -> x
Connections:
- net GND: now also C2.1, C3.1, D1.2 (A), U2.2 (GND), U3.2 (GND)
- net LN: now also U2.6; no longer U1.48 (A4)
- net LP: now also U2.4; no longer U1.47 (A3)
- net RN: now also U3.6; no longer U1.27 (K14)
- net RP: now also U3.4; no longer U1.26 (L14)
- net +5V: now reaches D2.2 (A)
- net +5V: now also D1.1 (K)
- new net: U1.27 (K14), U3.1
- new net: U1.26 (L14), U3.3
- new net: U1.47 (A3), U2.3
- new net: U1.48 (A4), U2.1
- new net +3.3V: C2.2, C3.2, U2.5 (VCC), U3.5 (VCC)
Other:
- added sheet Power supplies (power_supplies_sch.kicad_sch)
- added sheet output (output.kicad_sch)

Commit message: Distortion reduction
Connections:
- net +3.3V: now also SW1.1, SW1.2, SW1.3, SW1.4, SW1.5, SW1.6, SW1.7, SW1.8
- new net: C1.2, D2.1 (K), U1.24 (VU)
Changed lines of the file:
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@@
-	)
-	(junction
-		(at 80.01 72.39)
-		(diameter 0)
-		(color 0 0 0 0)
 	)
 	(junction
@@
 	)
 	(junction
+		(at 59.69 45.72)
+		(diameter 0)
+		(color 0 0 0 0)
+	)
+	(junction
 		(at 227.33 71.12)
 		(diameter 0)
@@
 		(color 0 0 0 0)
 	)
-	(junction
-		(at 59.69 63.5)
-		(diameter 0)
-		(color 0 0 0 0)
-	)
 	(no_connect
 		(at 110.49 64.77)
@@
 	(wire
 		(pts
-			(xy 59.69 76.2) (xy 80.01 76.2)
-		)
-		(stroke
-			(width 0)
-			(type default)
-		)
-	)
-	(wire
-		(pts
 			(xy 110.49 31.75) (xy 130.81 31.75)
 		)
@@
 	(wire
 		(pts
+			(xy 59.69 43.18) (xy 59.69 45.72)
+		)
+		(stroke
+			(width 0)
+			(type default)
+		)
+	)
+	(wire
+		(pts
 			(xy 48.26 29.21) (xy 72.39 29.21)
 		)
@@
 	(wire
 		(pts
-			(xy 76.2 72.39) (xy 80.01 72.39)
-		)
-		(stroke
-			(width 0)
-			(type default)
-		)
-	)
-	(wire
-		(pts
 			(xy 48.26 26.67) (xy 64.77 26.67)
 		)
@@
 	(wire
 		(pts
-			(xy 80.01 76.2) (xy 80.01 72.39)
-		)
-		(stroke
-			(width 0)
-			(type default)
-		)
-	)
-	(wire
-		(pts
 			(xy 72.39 26.67) (xy 86.36 26.67)
 		)
@@
 	(wire
 		(pts
-			(xy 59.69 63.5) (xy 59.69 76.2)
-		)
-		(stroke
-			(width 0)
-			(type default)
-		)
-	)
-	(wire
-		(pts
 			(xy 154.94 50.8) (xy 160.02 50.8)
 		)
@@
 	(wire
 		(pts
-			(xy 80.01 72.39) (xy 83.82 72.39)
+			(xy 76.2 72.39) (xy 83.82 72.39)
 		)
 		(stroke
@@
 					(unit 1)
 				)
+			)
+		)
+	)
+	(symbol
+		(lib_id "power:+3.3V")
+		(at 59.69 43.18 0)
+		(unit 1)
+		(body_style 1)
+		(exclude_from_sim no)
+		(in_bom yes)
+		(on_board yes)
+		(in_pos_files yes)
+		(dnp no)
+		(fields_autoplaced yes)
+		(property "Reference" "#PWR027"
+			(at 59.69 46.99 0)
+			(hide yes)
+			(show_name no)
+			(do_not_autoplace no)
+			(effects
+				(font
+					(size 1.27 1.27)
+				)
+			)
+		)
+		(property "Value" "+3.3V"
+			(at 59.69 38.1 0)
+			(show_name no)
+			(do_not_autoplace no)
+			(effects
+				(font
+					(size 1.27 1.27)
+				)
+			)
+		)
+		(property "Footprint" ""
+			(at 59.69 43.18 0)
+			(hide yes)
+			(show_name no)
+			(do_not_autoplace no)
+			(effects
+				(font
+					(size 1.27 1.27)
+				)
+			)
+		)
+		(property "Datasheet" ""
+			(at 59.69 43.18 0)
+			(hide yes)
+			(show_name no)
+			(do_not_autoplace no)
+			(effects
+				(font
+					(size 1.27 1.27)
+				)
+			)
+		)
+		(property "Description" "Power symbol creates a global label with name \"+3.3V\""
+			(at 59.69 43.18 0)
+			(hide yes)
+			(show_name no)
+			(do_not_autoplace no)
+			(effects
+				(font
+					(size 1.27 1.27)
+				)
+			)
+		)
+		(pin "1"
+		)
+		(instances
+			(project "dac-ng"
+				(path "/b8959107-fd4f-4873-b1a7-58431a0115ac"
+					(reference "#PWR027")
+					(unit 1)
+				)
