File: kicad/dac-ng/dac-ng.kicad_pcb (KiCad board)
At the start: 4 copper layers, 91.4 x 81.3 mm, 50 parts, among them J1 OUTPUT, J2 Conn_01x03_Pin, J3 Conn_01x08_Pin, J4 I2S_IN, SW1 SW_DIP_x08, U1 CMOD S7, U2 NE5532, U3 NE5532, U4 LM317_TO-220

Commit message: First run of v2.0
Parts:
- removed D3, D4: 1N4004, Diode_THT:D_DO-41_SOD81_P10.16mm_Horizontal
- removed the H2 at (148.6, 62.2)
- removed the J1 at (144.8, 89.0)
- removed the J2 at (144.8, 98.5)
- added C17: 680p, Capacitor_SMD:C_0603_1608Metric_Pad1.08x0.95mm_HandSolder, F.Cu at (112.8, 72.6)
- added C18: 680p, Capacitor_SMD:C_0603_1608Metric_Pad1.08x0.95mm_HandSolder, F.Cu at (112.8, 66.5)
- added C19: 680p, Capacitor_SMD:C_0603_1608Metric_Pad1.08x0.95mm_HandSolder, F.Cu at (112.3, 127.7)
- added C20: 680p, Capacitor_SMD:C_0603_1608Metric_Pad1.08x0.95mm_HandSolder, F.Cu at (112.3, 120.6)
- added C21: 680p, Capacitor_SMD:C_0603_1608Metric_Pad1.08x0.95mm_HandSolder, F.Cu at (121.1, 69.6)
- added C22: 680p, Capacitor_SMD:C_0603_1608Metric_Pad1.08x0.95mm_HandSolder, F.Cu at (120.8, 124.1)
- added C23: 100n, Capacitor_SMD:C_0603_1608Metric_Pad1.08x0.95mm_HandSolder, F.Cu at (131.1, 127.2)
- added C24: 100n, Capacitor_SMD:C_0603_1608Metric_Pad1.08x0.95mm_HandSolder, F.Cu at (135.2, 119.1)
- added C25: 680p, Capacitor_SMD:C_0603_1608Metric_Pad1.08x0.95mm_HandSolder, F.Cu at (121.1, 72.6)
- added C26: 680p, Capacitor_SMD:C_0603_1608Metric_Pad1.08x0.95mm_HandSolder, F.Cu at (121.1, 66.5)
- added C27: 680p, Capacitor_SMD:C_0603_1608Metric_Pad1.08x0.95mm_HandSolder, F.Cu at (120.8, 127.7)
- added C28: 680p, Capacitor_SMD:C_0603_1608Metric_Pad1.08x0.95mm_HandSolder, F.Cu at (120.8, 120.6)
- added C29: 180p, Capacitor_SMD:C_0603_1608Metric_Pad1.08x0.95mm_HandSolder, F.Cu at (135.1, 73.2)
- added C30: 180p, Capacitor_SMD:C_0603_1608Metric_Pad1.08x0.95mm_HandSolder, F.Cu at (135.2, 127.2)
- added C31: 180p, Capacitor_SMD:C_0603_1608Metric_Pad1.08x0.95mm_HandSolder, F.Cu at (131.1, 65.0)
- added C32: 180p, Capacitor_SMD:C_0603_1608Metric_Pad1.08x0.95mm_HandSolder, F.Cu at (131.1, 119.1)
- added C33: 10u, Capacitor_SMD:C_0805_2012Metric, F.Cu at (120.7, 97.3)
- added C34: 10u, Capacitor_SMD:C_0805_2012Metric, F.Cu at (120.7, 109.2)
- added C35: 1u, Capacitor_SMD:C_0603_1608Metric, F.Cu at (116.6, 79.5)
- added H4: MountingHole, MountingHole:MountingHole_3.2mm_M3, F.Cu at (144.8, 136.1)
- added J3: 7V UNREG, Connector_JST:JST_PH_B2B-PH-K_1x02_P2.00mm_Vertical, F.Cu at (119.9, 83.4)
- added J4: ANALOG PWR, Connector_JST:JST_PH_B3B-PH-K_1x03_P2.00mm_Vertical, F.Cu at (122.2, 105.3)
- added J5: AUDIO OUT, Custom:SWITCHCRAFT_PJRAN2X1U01AUX, F.Cu at (148.2, 95.4)
- added R18: 1.8k, Resistor_SMD:R_0603_1608Metric_Pad0.98x0.95mm_HandSolder, F.Cu at (125.5, 68.1)
- added R19: 1.8k, Resistor_SMD:R_0603_1608Metric_Pad0.98x0.95mm_HandSolder, F.Cu at (125.5, 71.1)
- added R20: 15k, Resistor_SMD:R_0603_1608Metric_Pad0.98x0.95mm_HandSolder, F.Cu at (125.5, 74.2)
- added R21: 15k, Resistor_SMD:R_0603_1608Metric_Pad0.98x0.95mm_HandSolder, F.Cu at (125.0, 119.1)
- added R22: 1.8k, Resistor_SMD:R_0603_1608Metric_Pad0.98x0.95mm_HandSolder, F.Cu at (125.0, 122.1)
- added R23: 1.8k, Resistor_SMD:R_0603_1608Metric_Pad0.98x0.95mm_HandSolder, F.Cu at (125.0, 125.7)
- added R24: 15k, Resistor_SMD:R_0603_1608Metric_Pad0.98x0.95mm_HandSolder, F.Cu at (125.0, 128.7)
- added R25: 1k, Resistor_SMD:R_0603_1608Metric_Pad0.98x0.95mm_HandSolder, F.Cu at (140.2, 65.5)
- added R26: 1k, Resistor_SMD:R_0603_1608Metric_Pad0.98x0.95mm_HandSolder, F.Cu at (140.2, 71.6)
- added R27: 1k, Resistor_SMD:R_0603_1608Metric_Pad0.98x0.95mm_HandSolder, F.Cu at (139.7, 119.6)
- added R28: 1k, Resistor_SMD:R_0603_1608Metric_Pad0.98x0.95mm_HandSolder, F.Cu at (139.7, 126.7)
- added R29: 50, Resistor_SMD:R_0603_1608Metric_Pad0.98x0.95mm_HandSolder, F.Cu at (140.2, 68.6)
- added R30: 50, Resistor_SMD:R_0603_1608Metric_Pad0.98x0.95mm_HandSolder, F.Cu at (139.7, 123.1)
- added R31: 1k, Resistor_SMD:R_0603_1608Metric_Pad0.98x0.95mm_HandSolder, F.Cu at (116.8, 89.4)
- added U5: TPS7A39, Package_SON:Texas_S-PVSON-N10_ThermalVias, F.Cu at (112.6, 103.5)
- added U6: LT3045xDD, Package_DFN_QFN:DFN-10-1EP_3x3mm_P0.5mm_EP1.65x2.38mm, F.Cu at (113.4, 89.5)
- added U7: OPA1612AxD, Package_SO:SOIC-8_5.3x5.3mm_P1.27mm, F.Cu at (133.1, 69.1)
- added U8: OPA1612AxD, Package_SO:SOIC-8_5.3x5.3mm_P1.27mm, F.Cu at (132.6, 123.1)
- C1, C13, C14, C3: value 47p -> 100n; footprint Custom:C_Rect_L7.2mm_W3.0mm_P5.00mm_FKS2_FKP2_MKS2_MKP2_HandSolder -> Capacitor_SMD:C_0603_1608Metric_Pad1.08x0.95mm_HandSolder
- C10: footprint Custom:C_Rect_L7.2mm_W3.0mm_P5.00mm_FKS2_FKP2_MKS2_MKP2_HandSolder -> Capacitor_SMD:C_0603_1608Metric_Pad1.08x0.95mm_HandSolder
- C11, C12: value 100n -> 22u; footprint Custom:C_Rect_L7.2mm_W3.0mm_P5.00mm_FKS2_FKP2_MKS2_MKP2_HandSolder -> Capacitor_Tantalum_SMD:CP_EIA-3216-10_Kemet-I_HandSolder
- C15: value 10u -> 680p; footprint Capacitor_THT:CP_Radial_D8.0mm_P5.00mm -> Capacitor_SMD:C_0603_1608Metric_Pad1.08x0.95mm_HandSolder
- C16: value 100n -> 680p; footprint Custom:C_Rect_L7.2mm_W3.0mm_P5.00mm_FKS2_FKP2_MKS2_MKP2_HandSolder -> Capacitor_SMD:C_0603_1608Metric_Pad1.08x0.95mm_HandSolder
- C2: value 100p -> 100n; footprint Custom:C_Rect_L7.2mm_W3.0mm_P5.00mm_FKS2_FKP2_MKS2_MKP2_HandSolder -> Capacitor_SMD:C_0603_1608Metric_Pad1.08x0.95mm_HandSolder
- C4: value 47p -> 10u; footprint Custom:C_Rect_L7.2mm_W3.0mm_P5.00mm_FKS2_FKP2_MKS2_MKP2_HandSolder -> Capacitor_SMD:C_0805_2012Metric
- C5: value 100p -> 10n; footprint Custom:C_Rect_L7.2mm_W3.0mm_P5.00mm_FKS2_FKP2_MKS2_MKP2_HandSolder -> Capacitor_SMD:C_0603_1608Metric_Pad1.08x0.95mm_HandSolder
- C6: value 100p -> 22u; footprint Custom:C_Rect_L7.2mm_W3.0mm_P5.00mm_FKS2_FKP2_MKS2_MKP2_HandSolder -> Capacitor_Tantalum_SMD:CP_EIA-3216-10_Kemet-I_HandSolder
- C7: value 100p -> 10u; footprint Custom:C_Rect_L7.2mm_W3.0mm_P5.00mm_FKS2_FKP2_MKS2_MKP2_HandSolder -> Capacitor_SMD:C_0805_2012Metric
- C8: value 47p -> 10n; footprint Custom:C_Rect_L7.2mm_W3.0mm_P5.00mm_FKS2_FKP2_MKS2_MKP2_HandSolder -> Capacitor_SMD:C_0603_1608Metric_Pad1.08x0.95mm_HandSolder
- C9: value 100n -> 10n; footprint Custom:C_Rect_L7.2mm_W3.0mm_P5.00mm_FKS2_FKP2_MKS2_MKP2_HandSolder -> Capacitor_SMD:C_0603_1608Metric_Pad1.08x0.95mm_HandSolder
- D1: value SB140 -> CDBU70; footprint Diode_THT:D_DO-41_SOD81_P10.16mm_Horizontal -> Diode_SMD:D_0603_1608Metric
- D2: value 1N4004 -> CDBU70; footprint Diode_THT:D_DO-41_SOD81_P10.16mm_Horizontal -> Diode_SMD:D_0603_1608Metric
- R1, R2: value 10k -> 100; footprint Custom:R_Axial_DIN0204_L3.6mm_D1.6mm_P7.62mm_Horizontal_HandSolder -> Resistor_SMD:R_0603_1608Metric_Pad0.98x0.95mm_HandSolder
- R10, R9: value 220 -> 2.2k; footprint Custom:R_Axial_DIN0204_L3.6mm_D1.6mm_P7.62mm_Horizontal_HandSolder -> Resistor_SMD:R_0603_1608Metric_Pad0.98x0.95mm_HandSolder
- R11: value 6.8k -> 2.2k; footprint Custom:R_Axial_DIN0204_L3.6mm_D1.6mm_P7.62mm_Horizontal_HandSolder -> Resistor_SMD:R_0603_1608Metric_Pad0.98x0.95mm_HandSolder
- R12: value 4.7k -> 2.2k; footprint Custom:R_Axial_DIN0204_L3.6mm_D1.6mm_P7.62mm_Horizontal_HandSolder -> Resistor_SMD:R_0603_1608Metric_Pad0.98x0.95mm_HandSolder
- R13, R14: value 10k -> 2.2k; footprint Custom:R_Axial_DIN0204_L3.6mm_D1.6mm_P7.62mm_Horizontal_HandSolder -> Resistor_SMD:R_0603_1608Metric_Pad0.98x0.95mm_HandSolder
- R15, R16: value 100 -> 2.2k; footprint Custom:R_Axial_DIN0204_L3.6mm_D1.6mm_P7.62mm_Horizontal_HandSolder -> Resistor_SMD:R_0603_1608Metric_Pad0.98x0.95mm_HandSolder
- R17: value 100 -> 15k; footprint Custom:R_Axial_DIN0204_L3.6mm_D1.6mm_P7.62mm_Horizontal_HandSolder -> Resistor_SMD:R_0603_1608Metric_Pad0.98x0.95mm_HandSolder
- R3: value 6.8k -> 100; footprint Custom:R_Axial_DIN0204_L3.6mm_D1.6mm_P7.62mm_Horizontal_HandSolder -> Resistor_SMD:R_0603_1608Metric_Pad0.98x0.95mm_HandSolder
- R4: value 6.8k -> 33.2k; footprint Custom:R_Axial_DIN0204_L3.6mm_D1.6mm_P7.62mm_Horizontal_HandSolder -> Resistor_SMD:R_0603_1608Metric_Pad0.98x0.95mm_HandSolder
- R5: value 4.7k -> 90.9k; footprint Custom:R_Axial_DIN0204_L3.6mm_D1.6mm_P7.62mm_Horizontal_HandSolder -> Resistor_SMD:R_0603_1608Metric_Pad0.98x0.95mm_HandSolder
- R6, R7: value 4.7k -> 10k; footprint Custom:R_Axial_DIN0204_L3.6mm_D1.6mm_P7.62mm_Horizontal_HandSolder -> Resistor_SMD:R_0603_1608Metric_Pad0.98x0.95mm_HandSolder
- R8: value 6.8k -> 100k; footprint Custom:R_Axial_DIN0204_L3.6mm_D1.6mm_P7.62mm_Horizontal_HandSolder -> Resistor_SMD:R_0603_1608Metric_Pad0.98x0.95mm_HandSolder
- U2, U3: value NE5532 -> 74LVC2G34; footprint Package_DIP:DIP-8_W7.62mm -> Package_TO_SOT_SMD:SOT-363_SC-70-6
- U4: value LM317_TO-220 -> TPS7A2050PDBV; footprint Package_TO_SOT_THT:TO-220-3_Vertical -> Package_TO_SOT_SMD:SOT-23-5
- moved R15 75.8 mm to (116.4, 127.7)
- moved H3 74.0 mm to (144.8, 62.0)
- moved R16 67.0 mm to (116.5, 120.6)
- moved R13 58.5 mm to (116.8, 72.6)
- moved R3 56.5 mm to (79.8, 75.4)
- moved C3 55.4 mm to (104.7, 126.2)
- moved C14 55.0 mm to (131.1, 73.2)
- moved R17 54.5 mm to (125.5, 65.0)
- moved C1 53.7 mm to (106.7, 116.2), turned to 0 degrees
- moved R14 53.2 mm to (116.7, 66.5)
- moved C13 52.6 mm to (135.1, 65.0), turned to 0 degrees
- moved C8 37.6 mm to (108.2, 108.2), turned to 180 degrees
- moved C9 37.3 mm to (108.2, 97.0)
- moved C12 36.8 mm to (113.3, 99.1)
- moved C7 35.6 mm to (108.7, 91.6), turned to 180 degrees
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- renumbered H4 to H2, J4 to J1, J3 to J2
Connections:
- C1 pad 1: Net-(C1-Pad1) -> GND
- C1 pad 2: Net-(U2A--) -> Net-(D2-K)
- C10 pad 1: GND -> +3.3V
- C10 pad 2: -12V -> GND
- C11 pad 1: GND -> +12V
- C11 pad 2: +12V -> GND
- C13 pad 1: Net-(C13-Pad1) -> GND
- C13 pad 2: Net-(U3A--) -> +12V
- C14 pad 1: Net-(C14-Pad1) -> GND
- C14 pad 2: ROUT -> -12V
- C15 pad 1: Net-(D3-A) -> Net-(C15-Pad1)
- C15 pad 2: GND -> Net-(C15-Pad2)
- C16 pad 1: GND -> Net-(C16-Pad1)
- C16 pad 2: Net-(D1-K) -> Net-(C16-Pad2)
- C2 pad 1: LN -> GND
- C2 pad 2: GND -> +3.3V
- C3 pad 1: Net-(U2B-+) -> GND
- C3 pad 2: GND -> +3.3V
- C4 pad 1: Net-(C4-Pad1) -> +5V
- C4 pad 2: LOUT -> GND
- C5 pad 1: LP -> Net-(U5-NR/SS)
- C6 pad 1: RN -> Net-(U6-SET)
- C7 pad 1: RP -> +3.3V
- C8 pad 1: Net-(U3B-+) -> +12V
- C8 pad 2: GND -> Net-(U5-FBP)
- C9 pad 1: GND -> Net-(U5-FBN)
- C9 pad 2: +12V -> -12V
- D1 pad 1: Net-(D1-K) -> +5V
- D1 pad 2: Net-(D1-A) -> GND
- D2 pad 1: Net-(D1-A) -> Net-(D2-K)
- D2 pad 2: GND -> +5V
- R1 pad 1: Net-(U2A--) -> /LRCLK
- R1 pad 2: Net-(C1-Pad1) -> Net-(U1-L1)
- R10 pad 1: GND -> LN
- R10 pad 2: Net-(D3-A) -> Net-(C15-Pad2)
- R11 pad 1: Net-(C14-Pad1) -> RP
- R11 pad 2: Net-(U3B-+) -> Net-(C16-Pad1)
- R12 pad 2: Net-(U3A--) -> Net-(C16-Pad2)
- R13 pad 1: GND -> Net-(C15-Pad1)
- R13 pad 2: Net-(U3A-+) -> Net-(C21-Pad1)
- R14 pad 1: Net-(U3A--) -> Net-(C15-Pad2)
- R14 pad 2: Net-(C13-Pad1) -> Net-(C21-Pad2)
- R15 pad 1: /LRCLK -> Net-(C16-Pad1)
- R15 pad 2: Net-(U1-L1) -> Net-(C22-Pad1)
- R16 pad 1: /BCLK -> Net-(C16-Pad2)
- R16 pad 2: Net-(U1-M4) -> Net-(C22-Pad2)
- R17 pad 1: /DATA -> Net-(C21-Pad1)
- R17 pad 2: Net-(U1-M3) -> Net-(C31-Pad2)
- R2 pad 1: GND -> /BCLK
- R2 pad 2: Net-(U2A-+) -> Net-(U1-M4)
- R3 pad 1: Net-(C1-Pad1) -> /DATA
- R3 pad 2: Net-(C4-Pad1) -> Net-(U1-M3)
- R4 pad 1: Net-(C4-Pad1) -> Net-(U6-SET)
- R4 pad 2: Net-(U2B-+) -> GND
- R5 pad 1: LP -> +12V
- R5 pad 2: Net-(U2A-+) -> Net-(U5-FBP)
- R6 pad 1: LN -> GND
- R6 pad 2: Net-(U2A--) -> Net-(U5-FBP)
- R7 pad 1: RP -> Net-(U5-FBN)
- R7 pad 2: Net-(U3A-+) -> Net-(U5-BUF)
- R8 pad 1: Net-(C13-Pad1) -> Net-(U5-FBN)
- R8 pad 2: Net-(C14-Pad1) -> -12V
- R9 pad 1: Net-(D3-A) -> LP
- R9 pad 2: Net-(D1-A) -> Net-(C15-Pad1)
- SW1 pad 1: Net-(D1-K) -> Net-(D2-K)
- SW1 pad 2: Net-(D1-K) -> Net-(D2-K)
- SW1 pad 3: Net-(D1-K) -> Net-(D2-K)
- SW1 pad 4: Net-(D1-K) -> Net-(D2-K)
- SW1 pad 5: Net-(D1-K) -> Net-(D2-K)
- SW1 pad 6: Net-(D1-K) -> Net-(D2-K)
- SW1 pad 7: Net-(D1-K) -> Net-(D2-K)
- SW1 pad 8: Net-(D1-K) -> Net-(D2-K)
- U1 pad 24: Net-(D1-K) -> Net-(D2-K)
- U1 pad 26: RP -> Net-(U1-L14)
- U1 pad 27: RN -> Net-(U1-K14)
- U1 pad 47: LP -> Net-(U1-A3)
- U1 pad 48: LN -> Net-(U1-A4)
- U2 pad 1: Net-(C1-Pad1) -> Net-(U1-A4)
- U2 pad 2: Net-(U2A--) -> GND
- U2 pad 3: Net-(U2A-+) -> Net-(U1-A3)
- U2 pad 4: -12V -> LP
- U2 pad 5: Net-(U2B-+) -> +3.3V
- U2 pad 6: LOUT -> LN
- U3 pad 1: Net-(C13-Pad1) -> Net-(U1-K14)
- U3 pad 2: Net-(U3A--) -> GND
- U3 pad 3: Net-(U3A-+) -> Net-(U1-L14)
- U3 pad 4: -12V -> RP
- U3 pad 5: Net-(U3B-+) -> +3.3V
- U3 pad 6: ROUT -> RN
- U4 pad 1: Net-(D3-A) -> Net-(J3-Pin_2)
- U4 pad 2: Net-(D1-A) -> GND
- U4 pad 3: +12V -> Net-(J3-Pin_2)
Routing:
- net Net-(D1-K): track 106.4 -> 0.00 mm
- net +3.3V: track 0.00 -> 83.4 mm, vias 0 -> 5
- net Net-(D2-K): track 0.00 -> 63.5 mm
- net +5V: track 0.00 -> 56.9 mm
- net ROUT: track 50.5 -> 0.00 mm
- net Net-(D1-A): track 45.8 -> 0.00 mm
- net LOUT: track 37.3 -> 0.00 mm
- net Net-(D3-A): track 30.7 -> 0.00 mm
- net Net-(J5-Pad2_A): track 0.00 -> 25.9 mm
- net Net-(C13-Pad1): track 24.5 -> 0.00 mm
- net Net-(C1-Pad1): track 24.5 -> 0.00 mm
- net Net-(J5-Pad2_B): track 0.00 -> 24.1 mm
- net -12V: track 100.2 -> 77.5 mm, vias 1 -> 4
- net /Power supplies/+15V: track 0.00 -> 22.7 mm
- net Net-(U8B--): track 0.00 -> 22.2 mm, vias 0 -> 2
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Other:
- board size 91.4 x 81.3 mm -> 81 x 81.3 mm
- board text added: "+15V"
- board text added: "-15V"
- board text added: "7-9V"
- board text added: "The ToyDAC - by NJSwede v 2.0 / Jun 2026"
- board text removed: "+12V"
- board text removed: "-12V"
- board text removed: "OUTPUT"
- board text removed: "ToyDAC Experiment Platform"

Commit message: WIP
Connections:
- C29 pad 2: Net-(U7B--) -> Net-(C29-Pad2)
- C30 pad 2: Net-(U8B--) -> Net-(C30-Pad2)
- R20 pad 2: Net-(R20-Pad2) -> Net-(C29-Pad2)
- R24 pad 2: Net-(R24-Pad2) -> Net-(C30-Pad2)
- R26 pad 1: Net-(R20-Pad2) -> Net-(C29-Pad2)
- R28 pad 1: Net-(R24-Pad2) -> Net-(C30-Pad2)
- R29 pad 1: Net-(U7B--) -> Net-(C29-Pad2)
- R30 pad 1: Net-(U8B--) -> Net-(C30-Pad2)
- SW1 pad 1: Net-(D2-K) -> +3.3V
- SW1 pad 2: Net-(D2-K) -> +3.3V
- SW1 pad 3: Net-(D2-K) -> +3.3V
- SW1 pad 4: Net-(D2-K) -> +3.3V
- SW1 pad 5: Net-(D2-K) -> +3.3V
- SW1 pad 6: Net-(D2-K) -> +3.3V
- SW1 pad 7: Net-(D2-K) -> +3.3V
- SW1 pad 8: Net-(D2-K) -> +3.3V
- U7 pad 7: Net-(U7B--) -> Net-(C29-Pad2)
- U8 pad 7: Net-(U8B--) -> Net-(C30-Pad2)
Routing:
- net +3.3V: track 83.4 -> 137.2 mm
- net Net-(D2-K): track 63.5 -> 30.2 mm
- net Net-(C30-Pad2): track 0.00 -> 24.6 mm, vias 0 -> 2
- net Net-(C29-Pad2): track 0.00 -> 24.0 mm, vias 0 -> 2
- net Net-(R20-Pad2): track 14.0 -> 0.00 mm
- net Net-(R24-Pad2): track 13.7 -> 0.00 mm
- net Net-(U8B--): track 22.2 -> 11.9 mm, vias 2 -> 0
- net Net-(U7B--): track 21.9 -> 12.2 mm, vias 2 -> 0
- net GND: vias 178 -> 179
