File: kicad/dac-ng/output.kicad_sch (KiCad schematic)
At the start: 45 parts, among them J5 AUDIO OUT, U7 OPA1612AxD, U8 OPA1612AxD

Commit message: Distortion reduction
Connections:
- net at R27.1, R28.2, U8.6 (-): now also C30.2, R30.1, U8.7
- net at R25.1, R26.2, U7.6 (-): now also C29.2, R29.1, U7.7
Changed lines of the file:
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@@
+	)
+	(junction
+		(at 193.04 127)
+		(diameter 0)
+		(color 0 0 0 0)
 	)
 	(junction
@@
 	)
 	(junction
+		(at 194.31 68.58)
+		(diameter 0)
+		(color 0 0 0 0)
+	)
+	(junction
 		(at 82.55 176.53)
 		(diameter 0)
@@
 	(wire
 		(pts
+			(xy 213.36 114.3) (xy 213.36 129.54)
+		)
+		(stroke
+			(width 0)
+			(type default)
+		)
+	)
+	(wire
+		(pts
 			(xy 96.52 184.15) (xy 96.52 189.23)
 		)
@@
 	(wire
 		(pts
+			(xy 193.04 114.3) (xy 213.36 114.3)
+		)
+		(stroke
+			(width 0)
+			(type default)
+		)
+	)
+	(wire
+		(pts
+			(xy 193.04 127) (xy 193.04 114.3)
+		)
+		(stroke
+			(width 0)
+			(type default)
+		)
+	)
+	(wire
+		(pts
 			(xy 185.42 90.17) (xy 185.42 76.2)
 		)
@@
 	(wire
 		(pts
+			(xy 194.31 57.15) (xy 213.36 57.15)
+		)
+		(stroke
+			(width 0)
+			(type default)
+		)
+	)
+	(wire
+		(pts
 			(xy 168.91 137.16) (xy 213.36 137.16)
 		)
@@
 	(wire
 		(pts
+			(xy 213.36 57.15) (xy 213.36 71.12)
+		)
+		(stroke
+			(width 0)
+			(type default)
+		)
+	)
+	(wire
+		(pts
 			(xy 175.26 116.84) (xy 175.26 118.11)
 		)
@@
 	(wire
 		(pts
+			(xy 194.31 68.58) (xy 195.58 68.58)
+		)
+		(stroke
+			(width 0)
+			(type default)
+		)
+	)
+	(wire
+		(pts
 			(xy 86.36 48.26) (xy 91.44 48.26)
 		)
@@
 	(wire
 		(pts
+			(xy 193.04 127) (xy 195.58 127)
+		)
+		(stroke
+			(width 0)
+			(type default)
+		)
+	)
+	(wire
+		(pts
 			(xy 91.44 48.26) (xy 91.44 63.5)
 		)
@@
 	(wire
 		(pts
-			(xy 185.42 127) (xy 195.58 127)
+			(xy 185.42 127) (xy 193.04 127)
 		)
 		(stroke
@@
 	(wire
 		(pts
+			(xy 194.31 68.58) (xy 194.31 57.15)
+		)
+		(stroke
+			(width 0)
+			(type default)
+		)
+	)
+	(wire
+		(pts
 			(xy 227.33 71.12) (xy 227.33 73.66)
 		)
@@
 	(wire
 		(pts
-			(xy 185.42 68.58) (xy 195.58 68.58)
-		)
-		(stroke
+			(xy 185.42 68.58) (xy 194.31 68.58)
+		)
+		(stroke

Commit message: WIP
Connections:
- net at R27.1, R28.2, U8.6 (-): no longer C30.2, R30.1, U8.7
- net at R20.2, R26.1: now also C29.2, R29.1, U7.7
- net at R25.1, R26.2, U7.6 (-): no longer C29.2, R29.1, U7.7
- net at R24.2, R28.1: now also C30.2, R30.1, U8.7
Changed lines of the file:
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@@
+	)
+	(junction
+		(at 185.42 90.17)
+		(diameter 0)
+		(color 0 0 0 0)
 	)
 	(junction
@@
 	)
 	(junction
-		(at 193.04 127)
-		(diameter 0)
-		(color 0 0 0 0)
-	)
-	(junction
 		(at 213.36 71.12)
 		(diameter 0)
@@
 	)
 	(junction
+		(at 185.42 148.59)
+		(diameter 0)
+		(color 0 0 0 0)
+	)
+	(junction
 		(at 134.62 77.47)
 		(diameter 0)
@@
 	)
 	(junction
+		(at 213.36 78.74)
+		(diameter 0)
+		(color 0 0 0 0)
+	)
+	(junction
 		(at 185.42 127)
 		(diameter 0)
@@
 	)
 	(junction
-		(at 194.31 68.58)
-		(diameter 0)
-		(color 0 0 0 0)
-	)
-	(junction
 		(at 82.55 176.53)
 		(diameter 0)
@@
 	)
 	(junction
+		(at 213.36 137.16)
+		(diameter 0)
+		(color 0 0 0 0)
+	)
+	(junction
 		(at 115.57 63.5)
 		(diameter 0)
@@
 	(wire
 		(pts
-			(xy 213.36 114.3) (xy 213.36 129.54)
-		)
-		(stroke
-			(width 0)
-			(type default)
-		)
-	)
-	(wire
-		(pts
 			(xy 96.52 184.15) (xy 96.52 189.23)
 		)
@@
 	(wire
 		(pts
-			(xy 193.04 114.3) (xy 213.36 114.3)
-		)
-		(stroke
-			(width 0)
-			(type default)
-		)
-	)
-	(wire
-		(pts
-			(xy 193.04 127) (xy 193.04 114.3)
-		)
-		(stroke
-			(width 0)
-			(type default)
-		)
-	)
-	(wire
-		(pts
 			(xy 185.42 90.17) (xy 185.42 76.2)
 		)
@@
 	(wire
 		(pts
-			(xy 194.31 57.15) (xy 213.36 57.15)
-		)
-		(stroke
-			(width 0)
-			(type default)
-		)
-	)
-	(wire
-		(pts
 			(xy 168.91 137.16) (xy 213.36 137.16)
 		)
@@
 	(wire
 		(pts
+			(xy 185.42 90.17) (xy 213.36 90.17)
+		)
+		(stroke
+			(width 0)
+			(type default)
+		)
+	)
+	(wire
+		(pts
 			(xy 102.87 148.59) (xy 91.44 148.59)
 		)
@@
 	(wire
 		(pts
+			(xy 213.36 90.17) (xy 213.36 78.74)
+		)
+		(stroke
+			(width 0)
+			(type default)
+		)
+	)
+	(wire
+		(pts
+			(xy 213.36 148.59) (xy 213.36 137.16)
+		)
+		(stroke
+			(width 0)
+			(type default)
+		)
+	)
+	(wire
+		(pts
 			(xy 171.45 59.69) (xy 175.26 59.69)
 		)
@@
 	(wire
 		(pts
-			(xy 213.36 57.15) (xy 213.36 71.12)
-		)
-		(stroke
-			(width 0)
-			(type default)
-		)
-	)
-	(wire
-		(pts
 			(xy 175.26 116.84) (xy 175.26 118.11)
 		)
@@
 	(wire
 		(pts
-			(xy 194.31 68.58) (xy 195.58 68.58)
+			(xy 185.42 68.58) (xy 195.58 68.58)
 		)
 		(stroke
@@
 	(wire
 		(pts
-			(xy 193.04 127) (xy 195.58 127)
+			(xy 185.42 127) (xy 195.58 127)
 		)
 		(stroke
@@
 	(wire
 		(pts
+			(xy 185.42 148.59) (xy 213.36 148.59)
+		)
+		(stroke
+			(width 0)
+			(type default)
+		)
+	)
+	(wire
+		(pts
 			(xy 175.26 58.42) (xy 175.26 59.69)
 		)
@@
 	(wire
 		(pts
-			(xy 185.42 127) (xy 193.04 127)
-		)
-		(stroke
-			(width 0)
-			(type default)
-		)
-	)
-	(wire
-		(pts
 			(xy 96.52 189.23) (xy 102.87 189.23)
 		)
@@
 	(wire
 		(pts
-			(xy 194.31 68.58) (xy 194.31 57.15)
-		)
-		(stroke
-			(width 0)
-			(type default)
-		)
-	)
-	(wire
-		(pts
 			(xy 227.33 71.12) (xy 227.33 73.66)
 		)
@@
 		)
 		(stroke
-			(width 0)
-			(type default)
-		)
-	)
-	(wire
-		(pts
-			(xy 185.42 68.58) (xy 194.31 68.58)
-		)
-		(stroke
